Commit message: Update mobile_base.xacro

File: ros2_ws/src/robot/urdf/mobile_base.xacro (robot description, xacro)
@@ -127,5 +127,5 @@
         <parent link="base_link"/>
         <child link="arm_link"/>
-        <origin xyz="0 0 ${base_height}" rpy="0 0 0"/>
+        <origin xyz="0 0 ${base_height + 0.05}" rpy="0 0 0"/>
         <axis xyz="0 1 0"/>
         <limit lower="-1.57"
@@ -184,5 +184,5 @@
         <parent link="base_link"/>
         <child link="lidar_link"/>
-        <origin xyz="0 0 ${base_height + 0.05}"/>
+        <origin xyz="0 0 ${base_height+0.025}"/>
     </joint>
     <link name="imu_link">
@@ -257,3 +257,49 @@
         </sensor>
     </gazebo>
+    <ros2_control name="RoverControl" type="system">
+        <hardware>
+            <plugin>gz_ros2_control/GazeboSimSystem</plugin>
+        </hardware>
+        <joint name="arm_joint">
+            <command_interface name="position"/>
+            <state_interface name="position"/>
+            <state_interface name="velocity"/>
+        </joint>
+    </ros2_control>
+    <gazebo>
+        <plugin filename="ignition-gazebo-diff-drive-system" name="ignition::gazebo::systems::DiffDrive">
+            <left_joint>base_left_wheel_joint</left_joint>
+            <right_joint>base_right_wheel_joint</right_joint>
+            <wheel_separation>0.45</wheel_separation>
+            <wheel_radius>0.1</wheel_radius>
+            <odom_publish_frequency>50</odom_publish_frequency>
+            <topic>cmd_vel</topic>
+            <publish_odom>true</publish_odom>
+            <publish_odom_tf>true</publish_odom_tf>
+            <publish_wheel_tf>true</publish_wheel_tf>
+            <left_wheel_frame>left_wheel_link</left_wheel_frame>
+            <right_wheel_frame>right_wheel_link</right_wheel_frame>
+            <frame_id>odom</frame_id>
+            <child_frame_id>base_footprint</child_frame_id>
+        </plugin>
+    </gazebo>
+    <gazebo>
+        <plugin filename="gz_ros2_control-system" name="gz_ros2_control::GazeboSimROS2ControlPlugin">
+        <parameters>$(find robot)/config/robot_controllers.yaml</parameters>
+        </plugin>
+    </gazebo>
+    <gazebo reference="caster_wheel_link">
+        <mu1>0.0</mu1>
+        <mu2>0.0</mu2>
+        <kp>1000000.0</kp>
+        <kd>1.0</kd>
+    </gazebo>
+    <gazebo reference="left_wheel_link">
+        <mu1>1.5</mu1>
+        <mu2>1.5</mu2>
+    </gazebo>
+    <gazebo reference="right_wheel_link">
+        <mu1>1.5</mu1>
+        <mu2>1.5</mu2>
+    </gazebo>
 </robot>
